File: Tomo/Tomo.kicad_pcb (KiCad board)
At the start: 2 copper layers, 2 parts, among them U1 ADG1408YRUZ, U2 ADG1408YRUZ

Commit message: TomoV1
Parts:
- added BT1: Battery_Cell, Connector_PinHeader_2.54mm:PinHeader_1x02_P2.54mm_Vertical, F.Cu at (115.0, 103.0)
- added J1: Conn_01x02, Connector_PinSocket_2.54mm:PinSocket_1x02_P2.54mm_Vertical, F.Cu at (62.0, 78.0)
- added J2: Conn_01x02, Connector_PinSocket_2.54mm:PinSocket_1x02_P2.54mm_Vertical, F.Cu at (62.0, 30.0)
- added J3: Conn_01x03, Connector_PinSocket_2.54mm:PinSocket_1x03_P2.54mm_Vertical, F.Cu at (59.5, 36.0)
- added J4: Conn_01x08, Connector_PinSocket_2.54mm:PinSocket_1x08_P2.54mm_Vertical, F.Cu at (38.0, 51.1)
- added J5: Conn_01x03, Connector_PinSocket_2.54mm:PinSocket_1x03_P2.54mm_Vertical, F.Cu at (59.5, 85.0)
- added J6: Conn_01x08, Connector_PinSocket_2.54mm:PinSocket_1x08_P2.54mm_Vertical, F.Cu at (38.0, 98.0)
- added J7: Conn_01x04, Connector_PinHeader_2.54mm:PinHeader_1x04_P2.54mm_Vertical, F.Cu at (115.0, 80.8)
- added R1: 10k, Resistor_SMD:R_0603_1608Metric, F.Cu at (75.0, 80.0)
- added R2: 10k, Resistor_SMD:R_0603_1608Metric, F.Cu at (101.0, 76.2)
- added R3: 10k, Resistor_SMD:R_0603_1608Metric, F.Cu at (106.0, 76.0)
- added U3: AD5933, Package_SO:SSOP-16_5.3x6.2mm_P0.65mm, F.Cu at (91.0, 81.0)
- moved U2 64.5 mm to (62.5, 99.0)
- moved U1 48.8 mm to (62.5, 52.0)
Connections:
- U1 pad 1: unconnected-(U1-Pad1) -> Net-(J3-Pad1)
- U1 pad 10: unconnected-(U1-Pad10) -> Net-(J4-Pad7)
- U1 pad 11: unconnected-(U1-Pad11) -> Net-(J4-Pad6)
- U1 pad 12: unconnected-(U1-Pad12) -> Net-(J4-Pad5)
- U1 pad 13: unconnected-(U1-Pad13) -> +5V
- U1 pad 14: unconnected-(U1-Pad14) -> GND
- U1 pad 15: unconnected-(U1-Pad15) -> Net-(J3-Pad3)
- U1 pad 16: unconnected-(U1-Pad16) -> Net-(J3-Pad2)
- U1 pad 2: unconnected-(U1-Pad2) -> Net-(J2-Pad1)
- U1 pad 3: unconnected-(U1-Pad3) -> GND
- U1 pad 4: unconnected-(U1-Pad4) -> Net-(J4-Pad1)
- U1 pad 5: unconnected-(U1-Pad5) -> Net-(J4-Pad2)
- U1 pad 6: unconnected-(U1-Pad6) -> Net-(J4-Pad3)
- U1 pad 7: unconnected-(U1-Pad7) -> Net-(J4-Pad4)
- U1 pad 8: unconnected-(U1-Pad8) -> /IN
- U1 pad 9: unconnected-(U1-Pad9) -> Net-(J4-Pad8)
- U2 pad 1: unconnected-(U2-Pad1) -> Net-(J5-Pad1)
- U2 pad 10: unconnected-(U2-Pad10) -> Net-(J6-Pad7)
- U2 pad 11: unconnected-(U2-Pad11) -> Net-(J6-Pad6)
- U2 pad 12: unconnected-(U2-Pad12) -> Net-(J6-Pad5)
- U2 pad 13: unconnected-(U2-Pad13) -> +5V
- U2 pad 14: unconnected-(U2-Pad14) -> GND
- U2 pad 15: unconnected-(U2-Pad15) -> Net-(J5-Pad3)
- U2 pad 16: unconnected-(U2-Pad16) -> Net-(J5-Pad2)
- U2 pad 2: unconnected-(U2-Pad2) -> Net-(J1-Pad1)
- U2 pad 3: unconnected-(U2-Pad3) -> GND
- U2 pad 4: unconnected-(U2-Pad4) -> Net-(J6-Pad1)
- U2 pad 5: unconnected-(U2-Pad5) -> Net-(J6-Pad2)
- U2 pad 6: unconnected-(U2-Pad6) -> Net-(J6-Pad3)
- U2 pad 7: unconnected-(U2-Pad7) -> Net-(J6-Pad4)
- U2 pad 8: unconnected-(U2-Pad8) -> /OUT
- U2 pad 9: unconnected-(U2-Pad9) -> Net-(J6-Pad8)
Routing:
- net /IN: track 0.00 -> 59.0 mm, vias 0 -> 2
- net /OUT: track 0.00 -> 58.7 mm, vias 0 -> 2
- net Net-(J4-Pad8): track 0.00 -> 33.4 mm
- net Net-(J6-Pad8): track 0.00 -> 33.3 mm
- net Net-(J4-Pad7): track 0.00 -> 32.6 mm
- net Net-(J6-Pad7): track 0.00 -> 32.6 mm
- net Net-(J4-Pad6): track 0.00 -> 31.8 mm
- net Net-(J6-Pad6): track 0.00 -> 31.8 mm
- net Net-(J4-Pad5): track 0.00 -> 31.2 mm
- net Net-(J6-Pad5): track 0.00 -> 31.1 mm
- net Net-(J2-Pad1): track 0.00 -> 25.8 mm
- net Net-(J1-Pad1): track 0.00 -> 24.0 mm
- net Net-(J4-Pad4): track 0.00 -> 23.7 mm
- net Net-(J6-Pad4): track 0.00 -> 23.7 mm
- net Net-(J4-Pad3): track 0.00 -> 23.0 mm
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- added copper zone on B.Cu, net +5V
- added copper zone on F.Cu, net GND
Other:
- board outline added: 100 x 100 mm
- board text added: "AD5933 ADG1608 Evaluation Board"
- board text added: "By 张庭梁 20211231 All Right Reserves"
