File: Tomo/Tomo.kicad_sch (KiCad schematic)
At the start: 15 parts, among them J1 Conn_01x02, J2 Conn_01x02, J3 Conn_01x03, J4 Conn_01x08, J5 Conn_01x03, J6 Conn_01x08, J7 Conn_01x04, U1 ADG1408YRUZ, U2 ADG1408YRUZ, U3 AD5933

Commit message: TomoV1
Parts:
- J7: footprint (none) -> Connector_PinHeader_2.54mm:PinHeader_1x04_P2.54mm_Vertical
Changed lines of the file:
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@@
     (property "Reference" "J7" (id 0) (at 182.88 53.34 0))
     (property "Value" "Conn_01x04" (id 1) (at 182.88 55.88 0))
-    (property "Footprint" "" (id 2) (at 182.88 64.77 0)
+    (property "Footprint" "Connector_PinHeader_2.54mm:PinHeader_1x04_P2.54mm_Vertical" (id 2) (at 182.88 64.77 0)
       (effects (font (size 1.27 1.27)) hide)
     )
@@
     )
     (path "/de7fd075-957c-46b2-bffb-645bde5fdae7"
-      (reference "J7") (unit 1) (value "Conn_01x04") (footprint "")
+      (reference "J7") (unit 1) (value "Conn_01x04") (footprint "Connector_PinHeader_2.54mm:PinHeader_1x04_P2.54mm_Vertical")
     )
     (path "/18084a95-067b-48a6-a95c-51150bff3631"
