File: HandGesturePCB/HandGesturePCB.kicad_sch (KiCad schematic)
At the start: 2 parts

Commit message: Update HandGesturePCB.kicad_sch
Parts:
- added BT?: Battery_Cell, Connector_PinHeader_2.54mm:PinHeader_1x02_P2.54mm_Vertical, symbol Device:Battery_Cell
- added D?: LED, symbol Device:LED
- added J? (x2): Conn_01x02, Connector_PinSocket_2.54mm:PinSocket_1x02_P2.54mm_Vertical, symbol Connector_Generic:Conn_01x02
- added J? (x2): Conn_01x08, Connector_PinHeader_2.54mm:PinHeader_1x08_P2.54mm_Vertical, symbol Connector_Generic:Conn_01x08
- added J?: Conn_01x04, Connector_PinHeader_2.54mm:PinHeader_1x04_P2.54mm_Vertical, symbol Connector_Generic:Conn_01x04
- added R? (x3): 10k, Resistor_SMD:R_0603_1608Metric, symbol Device:R
- added U?: 74HC4051, Package_SO:TSSOP-16_4.4x5mm_P0.65mm, symbol 74xx:74HC4051
- U?: footprint (none) -> Package_SO:TSSOP-16_4.4x5mm_P0.65mm
Connections:
- net +5V: now also U?.10 (AVDD1), U?.11 (AVDD2), U?.16 (VCC), U?.9 (DVDD), BT?.1 (+), D?.2 (A), J?.1 (Pin_1), J?.1 (Pin_1), R?.1, R?.1, U?.16 (VCC)
- net A0: now also J?.8 (Pin_8), U?.13 (A0)
- net A1: now also J?.7 (Pin_7), U?.14 (A1)
- net A2: now also J?.6 (Pin_6), U?.15 (A2)
- net A3: now also J?.5 (Pin_5), U?.12 (A3)
- net A4: now also J?.4 (Pin_4), U?.1 (A4)
- net A5: now also J?.3 (Pin_3), U?.5 (A5)
- net A6: now also J?.2 (Pin_2), U?.2 (A6)
- net A7: now also J?.1 (Pin_1), U?.4 (A7)
- net GND: now also U?.12 (DGND), U?.13 (AGND1), U?.14 (AGND2), U?.8 (MCLK), BT?.2 (-), D?.1 (K), J?.2 (Pin_2), J?.8 (Pin_8), U?.7 (VEE), U?.8 (GND)
- net SDA: now reaches U?.15 (SDA)
- net SDA: now also J?.3 (Pin_3), R?.2
- net SCL: now reaches U?.16 (SCL)
- net SCL: now also J?.4 (Pin_4), R?.2
- net at U?.4 (RFB): now also R?.2
- net IN: now reaches U?.5 (VIN)
- net IN: now also U?.3 (A), J?.1 (Pin_1), R?.1
- net OUT: now reaches U?.6 (VOUT)
- net OUT: now also J?.2 (Pin_2), U?.3 (A)
- net S01: now reaches U?.10 (S1)
- net S01: now also J?.3 (Pin_3)
- net S00: now reaches U?.11 (S0)
- net S00: now also J?.2 (Pin_2)
- net ENABLE: now reaches U?.6 (~{E})
- net ENABLE: now also J?.1 (Pin_1), J?.2 (Pin_2), U?.6 (~{E})
- net S02: now reaches U?.9 (S2)
- net S02: now also J?.4 (Pin_4)
- new net S10: J?.5 (Pin_5), U?.11 (S0)
- new net S11: J?.6 (Pin_6), U?.10 (S1)
- new net S12: J?.7 (Pin_7), U?.9 (S2)

Commit message: Update HandGesturePCB.kicad_sch
Parts:
- added R4: 200, Resistor_SMD:R_0603_1608Metric, symbol Device:R
- D1: renamed from D?; footprint (none) -> LED_SMD:LED_0603_1608Metric
- gave numbers to parts that had none: 12
Connections:
- net +5V: now also R4.1; no longer D1.2 (A)
- new net: D1.2 (A), R4.2
Other:
- moved on the sheet: BT1, D1, J1, J2, J3, J4, J5, R1, R2, R3, U1, U2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

Commit message: beginLayout
Parts:
- removed BT1: Battery_Cell, Connector_PinHeader_2.54mm:PinHeader_1x02_P2.54mm_Vertical, symbol Device:Battery_Cell
Changed lines of the file:
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@@
     (pin "1")
-  )
-  (symbol (lib_id "Device:Battery_Cell") (at 203.2 72.39 0) (unit 1)
-    (in_bom yes) (on_board yes) (fields_autoplaced)
-    (property "Reference" "BT1" (id 0) (at 207.01 69.0879 0)
-      (effects (font (size 1.27 1.27)) (justify left))
-    )
-    (property "Value" "Battery_Cell" (id 1) (at 207.01 71.6279 0)
-      (effects (font (size 1.27 1.27)) (justify left))
-    )
-    (property "Footprint" "Connector_PinHeader_2.54mm:PinHeader_1x02_P2.54mm_Vertical" (id 2) (at 203.2 70.866 90)
-      (effects (font (size 1.27 1.27)) hide)
-    )
-    (property "Datasheet" "~" (id 3) (at 203.2 70.866 90)
-      (effects (font (size 1.27 1.27)) hide)
-    )
-    (pin "1")
-    (pin "2")
   )
   (symbol (lib_id "Connector_Generic:Conn_01x02") (at 34.29 95.25 0) (unit 1)
@@
     (pin "9")
   )
-  (symbol (lib_id "power:+5V") (at 203.2 67.31 0) (unit 1)
-    (in_bom yes) (on_board yes)
-    (property "Reference" "#PWR0117" (id 0) (at 203.2 71.12 0)
-      (effects (font (size 1.27 1.27)) hide)
-    )
-    (property "Value" "+5V" (id 1) (at 200.66 63.5 0)
-      (effects (font (size 1.27 1.27)) (justify left))
-    )
-    (property "Footprint" "" (id 2) (at 203.2 67.31 0)
-      (effects (font (size 1.27 1.27)) hide)
-    )
-    (property "Datasheet" "" (id 3) (at 203.2 67.31 0)
-      (effects (font (size 1.27 1.27)) hide)
-    )
-    (pin "1")
-  )
   (symbol (lib_id "Connector_Generic:Conn_01x08") (at 34.29 71.12 0) (unit 1)
     (in_bom yes) (on_board yes) (fields_autoplaced)
@@
     (pin "1")
   )
-  (symbol (lib_id "power:GND") (at 203.2 74.93 0) (unit 1)
-    (in_bom yes) (on_board yes) (fields_autoplaced)
-    (property "Reference" "#PWR0114" (id 0) (at 203.2 81.28 0)
-      (effects (font (size 1.27 1.27)) hide)
-    )
-    (property "Value" "GND" (id 1) (at 205.74 76.1999 0)
-      (effects (font (size 1.27 1.27)) (justify left))
-    )
-    (property "Footprint" "" (id 2) (at 203.2 74.93 0)
-      (effects (font (size 1.27 1.27)) hide)
-    )
-    (property "Datasheet" "" (id 3) (at 203.2 74.93 0)
-      (effects (font (size 1.27 1.27)) hide)
-    )
-    (pin "1")
-  )
   (symbol (lib_id "power:+5V") (at 69.85 22.86 0) (unit 1)
     (in_bom yes) (on_board yes) (fields_autoplaced)
@@
       (reference "#PWR0113") (unit 1) (value "+5V") (footprint "")
     )
-    (path "/e9be6a11-97e0-4bce-a99c-caa58a26cd7d"
-      (reference "#PWR0114") (unit 1) (value "GND") (footprint "")
-    )
     (path "/37532192-ed7f-47fc-a78e-81dc6d31d5a2"
       (reference "#PWR0115") (unit 1) (value "GND") (footprint "")
@@
       (reference "#PWR0116") (unit 1) (value "+5V") (footprint "")
     )
-    (path "/87139ac4-ba87-4996-81d2-7a65ceeeb915"
-      (reference "#PWR0117") (unit 1) (value "+5V") (footprint "")
-    )
-    (path "/11e341bf-72a6-449c-853f-ff43b5daa225"
-      (reference "BT1") (unit 1) (value "Battery_Cell") (footprint "Connector_PinHeader_2.54mm:PinHeader_1x02_P2.54mm_Vertical")
-    )
     (path "/d2e18776-eb03-49f5-b099-f889f3fc3f7a"
