File: HandGesturePCB/HandGesturePCB.kicad_pcb (KiCad board)
At the start: 2 copper layers, 14 parts, among them J1 Conn_01x08, J2 Conn_01x08, J3 Conn_01x02, J4 Conn_01x02, J5 Conn_01x04, U1 74HC4051, U2 74HC4051, U3 AD5933

Commit message: beginLayout
Parts:
- removed BT1: Battery_Cell, Connector_PinHeader_2.54mm:PinHeader_1x02_P2.54mm_Vertical
- moved J5 120.0 mm to (23.0, 36.7)
- moved D1 113.5 mm to (34.0, 36.5), turned to 90 degrees
- moved R4 108.8 mm to (40.0, 36.5), turned to 90 degrees
- moved R2 102.1 mm to (34.0, 43.5), turned to -90 degrees
- moved R3 95.2 mm to (40.0, 43.5), turned to -90 degrees
- moved U3 68.7 mm to (59.0, 39.5), turned to 180 degrees
- moved R1 55.8 mm to (66.0, 41.5), turned to -90 degrees
- moved J3 50.0 mm to (102.0, 24.5)
- moved J4 47.3 mm to (71.0, 40.5), turned to 180 degrees
- moved U2 27.3 mm to (80.0, 32.5)
- moved J1 15.1 mm to (71.3, 21.5)
- moved U1 13.4 mm to (80.0, 46.5)
- moved J2 8.16 mm to (102.0, 34.1)

Commit message: Finish
Parts:
- turned R3 to 90 degrees
Routing:
- net GND: track 0.00 -> 213.0 mm, vias 0 -> 2
- net +5V: track 0.00 -> 177.4 mm, vias 0 -> 4
- net /ENABLE: track 0.00 -> 50.1 mm, vias 0 -> 2
- net /A3: track 0.00 -> 44.7 mm, vias 0 -> 1
- net /SCL: track 0.00 -> 35.0 mm
- net /SDA: track 0.00 -> 33.6 mm
- net /A7: track 0.00 -> 33.3 mm, vias 0 -> 2
- net /A5: track 0.00 -> 32.5 mm, vias 0 -> 3
- net /A1: track 0.00 -> 32.0 mm
- net /A2: track 0.00 -> 31.7 mm
- net /A0: track 0.00 -> 31.2 mm, vias 0 -> 2
- net /A6: track 0.00 -> 28.6 mm, vias 0 -> 2
- net /S11: track 0.00 -> 26.0 mm
- net /A4: track 0.00 -> 25.9 mm
- net /S12: track 0.00 -> 25.2 mm
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Other:
- board outline added: 100 x 100 mm
- board text added: "AD5933 CD74HC4051PWR Evaluation Board"
- board text added: "By TingliangZhang 20220314 Midnight"
